File: kicad/genbox.kicad_pcb (KiCad board)
At the start: 2 copper layers, 367 x 147.5 mm, 22 parts, among them SW15 SW_SPST, SW16 SW_SPST, SW17 SW_SPST, SW18 SW_SPST

Commit message: doubled trace width
Routing:
- net LEFT: track 185.0 -> 79.3 mm
- net RIGHT: track 68.8 -> 160.6 mm
- net DOWN: track 110.3 -> 72.2 mm, vias 0 -> 2
- net R2: track 270.6 -> 258.8 mm
- net S2: track 173.8 -> 164.6 mm, vias 1 -> 0
- net L1: track 263.6 -> 254.7 mm
- net S1: track 156.2 -> 149.2 mm, vias 1 -> 0
- net B2: track 239.0 -> 233.9 mm
- net L3: track 136.0 -> 131.3 mm
- net UP: track 44.8 -> 40.7 mm, vias 0 -> 2
- net R1: track 230.1 -> 226.5 mm
- net B1: track 221.9 -> 218.4 mm
- net R3: track 219.8 -> 216.8 mm
- net L2: track 284.4 -> 286.2 mm
- net A2: track 67.8 -> 66.1 mm
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Other:
- board text added: "original design by Genthus"

Commit message: pcb dimension changes
Parts:
- moved REF1 0.07 mm to (199.6, 77.0)
- moved REF2 0.07 mm to (199.6, 150.0)
Routing:
- net RIGHT: track 160.6 -> 156.0 mm
- net S1: track 149.2 -> 149.8 mm
Other:
- board size 367 x 147.5 mm -> 350.4 x 147.1 mm

Commit message: rework p1
Parts:
- removed REF1: MountingHole_4mm, MountingHole:MountingHole_4mm
- removed REF2: MountingHole_5mm, MountingHole:MountingHole_5mm
- removed RZ1: RP2040-Zero, RP2040-Zero-Kicad-main:RP2040-Zero
- added C1: C, Capacitor_SMD:C_0805_2012Metric_Pad1.18x1.45mm_HandSolder, F.Cu at (122.0, 114.6)
- added C10: C, Capacitor_SMD:C_0805_2012Metric_Pad1.18x1.45mm_HandSolder, F.Cu at (126.8, 123.7)
- added C11: C, Capacitor_SMD:C_0805_2012Metric_Pad1.18x1.45mm_HandSolder, F.Cu at (126.8, 126.7)
- added C12: C, Capacitor_SMD:C_0805_2012Metric_Pad1.18x1.45mm_HandSolder, F.Cu at (126.8, 129.7)
- added C13: C, Capacitor_SMD:C_0805_2012Metric_Pad1.18x1.45mm_HandSolder, F.Cu at (131.6, 114.6)
- added C14: C, Capacitor_SMD:C_0805_2012Metric_Pad1.18x1.45mm_HandSolder, F.Cu at (131.6, 117.6)
- added C15: C, Capacitor_SMD:C_0805_2012Metric_Pad1.18x1.45mm_HandSolder, F.Cu at (131.6, 120.7)
- added C2: C, Capacitor_SMD:C_0805_2012Metric_Pad1.18x1.45mm_HandSolder, F.Cu at (122.0, 117.6)
- added C3: C, Capacitor_SMD:C_0805_2012Metric_Pad1.18x1.45mm_HandSolder, F.Cu at (122.0, 120.7)
- added C4: C, Capacitor_SMD:C_0805_2012Metric_Pad1.18x1.45mm_HandSolder, F.Cu at (122.0, 123.7)
- added C5: C, Capacitor_SMD:C_0805_2012Metric_Pad1.18x1.45mm_HandSolder, F.Cu at (122.0, 126.7)
- added C6: C, Capacitor_SMD:C_0805_2012Metric_Pad1.18x1.45mm_HandSolder, F.Cu at (122.0, 129.7)
- added C7: C, Capacitor_SMD:C_0805_2012Metric_Pad1.18x1.45mm_HandSolder, F.Cu at (126.8, 114.6)
- added C8: C, Capacitor_SMD:C_0805_2012Metric_Pad1.18x1.45mm_HandSolder, F.Cu at (126.8, 117.6)
- added C9: C, Capacitor_SMD:C_0805_2012Metric_Pad1.18x1.45mm_HandSolder, F.Cu at (126.8, 120.7)
- added D1: SK6812, haku:SK6812-MINI-E_MX, B.Cu at (174.5, 79.1)
- added D10: SK6812, haku:SK6812-MINI-E_MX, B.Cu at (198.6, 97.8)
- added D11: SK6812, haku:SK6812-MINI-E_MX, B.Cu at (221.0, 68.0)
- added D12: SK6812, haku:SK6812-MINI-E_MX, B.Cu at (158.9, 83.8)
- added D13: SK6812, haku:SK6812-MINI-E_MX, B.Cu at (158.9, 88.4)
- added D14: SK6812, haku:SK6812-MINI-E_MX, B.Cu at (158.9, 93.0)
- added D2: SK6812, haku:SK6812-MINI-E_MX, B.Cu at (174.5, 83.8)
- added D3: SK6812, haku:SK6812-MINI-E_MX, B.Cu at (174.5, 88.4)
- added D4: SK6812, haku:SK6812-MINI-E_MX, B.Cu at (174.5, 93.0)
- added D5: SK6812, haku:SK6812-MINI-E_MX, B.Cu at (174.5, 97.6)
- added D6: SK6812, haku:SK6812-MINI-E_MX, B.Cu at (166.7, 79.1)
- added D7: SK6812, haku:SK6812-MINI-E_MX, B.Cu at (166.7, 83.8)
- added D8: SK6812, haku:SK6812-MINI-E_MX, B.Cu at (166.7, 88.4)
- added D9: SK6812, haku:SK6812-MINI-E_MX, B.Cu at (166.7, 93.0)
- added F1: Fuse, Fuse:Fuse_0805_2012Metric_Pad1.15x1.40mm_HandSolder, F.Cu at (171.2, 147.5)
- added J1: USB_A, Connector_USB:USB_A_Receptacle_GCT_USB1046, B.Cu at (114.3, 59.7)
- added R1: 10k, Resistor_SMD:R_0603_1608Metric_Pad0.98x0.95mm_HandSolder, F.Cu at (171.0, 135.3)
- added R2: 10k, Resistor_SMD:R_0603_1608Metric_Pad0.98x0.95mm_HandSolder, F.Cu at (171.0, 137.8)
- added R3: 10k, Resistor_SMD:R_0603_1608Metric_Pad0.98x0.95mm_HandSolder, F.Cu at (171.0, 140.3)
- added U1: DM-OLED096-636, DM-OLED096-636:MODULE_DM-OLED096-636, F.Cu at (74.9, 82.5)
- added U2: rp2040-zero, mcu:rp2040-zero-smd-pads, B.Cu at (184.0, 64.2)
- added U3: SN74LV1T34DBV, Package_TO_SOT_SMD:SOT-23-5, F.Cu at (171.4, 143.8)
- SW15, SW16, SW17, SW18: footprint Button_Switch_THT:SW_PUSH_6mm_H7.3mm -> Button_Switch_THT:SW_PUSH-12mm
- moved MX1 213.4 mm to (261.3, 62.0)
- moved MX6 181.5 mm to (241.2, 62.0)
- moved MX3 177.0 mm to (261.3, 102.3)
- moved MX5 172.6 mm to (261.3, 142.7)
- moved SW15 155.8 mm to (307.4, 31.8)
- moved MX4 153.1 mm to (261.3, 122.5)
- moved MX11 144.7 mm to (221.0, 62.0)
- moved MX14 141.8 mm to (221.0, 122.5)
- moved G*** 136.6 mm to (177.7, 298.3)
- moved SW16 132.7 mm to (307.4, 45.3)
- moved MX13 124.8 mm to (221.0, 102.3)
- moved MX2 123.4 mm to (261.3, 82.2)
- moved MX12 106.8 mm to (221.0, 82.2)
- moved MX10 97.6 mm to (241.2, 142.7)
- moved SW17 96.5 mm to (307.4, 58.9)
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Routing:
- net L2: track 286.2 -> 0.00 mm
- net R2: track 258.8 -> 0.00 mm
- net L1: track 254.7 -> 0.00 mm
- net B2: track 233.9 -> 0.00 mm
- net R1: track 226.5 -> 0.00 mm
- net B1: track 218.4 -> 0.00 mm
- net R3: track 216.8 -> 0.00 mm, vias 2 -> 0
- net B4: track 196.1 -> 0.00 mm
- net B3: track 178.5 -> 0.00 mm
- net S2: track 164.6 -> 0.00 mm
- net RIGHT: track 156.0 -> 0.00 mm
- net S1: track 149.8 -> 0.00 mm
- net L3: track 131.3 -> 0.00 mm, vias 2 -> 0
- net LEFT: track 79.3 -> 0.00 mm
- net DOWN: track 72.2 -> 0.00 mm, vias 2 -> 0
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- removed copper zone on B.Cu, net GND
Other:
- board size 350.4 x 147.1 mm -> 11.3 x 21 mm

Commit message: pcb rework complete
Parts:
- C1, C10, C11, C12, C13, C14, C15, C2, C3, C4, C5, C6, C7, C8, C9: value C -> 100nF; moved to B.Cu
- D1, D10, D11, D12, D13, D14, D2, D3, D4, D5, D6, D7, D8, D9: moved to F.Cu
- F1: value Fuse -> 1A; moved to B.Cu
- J1: footprint Connector_USB:USB_A_Receptacle_GCT_USB1046 -> Connector_USB:USB_A_Molex_67643_Horizontal; moved to F.Cu
- R1, R2, R3: value 10k -> 22Ω; moved to B.Cu
- SW15, SW16, SW17, SW18: footprint Button_Switch_THT:SW_PUSH-12mm -> haku:SW_PUSH-12mm_centered
- U1: footprint DM-OLED096-636:MODULE_DM-OLED096-636 -> haku:OLED-128x64
- U2: footprint mcu:rp2040-zero-smd-pads -> mcu:rp2040-zero-tht-pads
- U3: moved to B.Cu
- moved C5 260.1 mm to (382.0, 132.0), turned to 180 degrees
- moved C4 258.0 mm to (379.0, 101.0), turned to 180 degrees
- moved C6 233.1 mm to (355.0, 124.0), turned to 180 degrees
- moved C3 228.4 mm to (349.0, 96.0), turned to 180 degrees
- moved C2 204.2 mm to (325.0, 96.0), turned to 180 degrees
- moved C7 203.6 mm to (330.0, 127.0), turned to 180 degrees
- moved D5 198.1 mm to (371.5, 118.0), turned to 0 degrees
- moved D4 190.1 mm to (364.5, 91.9), turned to 0 degrees
- moved MX1 186.2 mm to (80.4, 105.7)
- moved G*** 181.3 mm to (197.0, 118.0)
- moved C8 181.0 mm to (307.0, 134.0), turned to 180 degrees
- moved D6 180.8 mm to (344.7, 110.7), turned to 0 degrees
- moved C15 168.8 mm to (300.0, 109.0), turned to 180 degrees
- moved D3 163.3 mm to (337.7, 84.6), turned to 0 degrees
- moved MX5 158.7 mm to (114.8, 81.8)
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Connections:
- U2 pad 1: S1 -> USBA D+
- U2 pad 10: L2 -> R3
- U2 pad 11: B3 -> B1
- U2 pad 12: B4 -> B3
- U2 pad 13: R1 -> B2
- U2 pad 14: L1 -> B4
- U2 pad 15: A1 -> R2
- U2 pad 16: A2 -> R1
- U2 pad 17: L3 -> S1
- U2 pad 18: R3 -> S2
- U2 pad 19: OLED SDA -> A1
- U2 pad 2: S2 -> USBA D-
- U2 pad 20: OLED SCL -> A2
- U2 pad 24: USBA D+ -> L2
- U2 pad 25: USBA D- -> L1
- U2 pad 3: UP -> OLED SCL
- U2 pad 4: DOWN -> OLED SDA
- U2 pad 5: RIGHT -> UP
- U2 pad 6: LEFT -> DOWN
- U2 pad 7: B1 -> LEFT
- U2 pad 8: B2 -> RIGHT
- U2 pad 9: R2 -> L3
Routing:
- net +5V: track 0.00 -> 1107.1 mm, vias 0 -> 12
- net L2: track 0.00 -> 184.6 mm, vias 0 -> 1
- net LEFT: track 0.00 -> 181.8 mm
- net L1: track 0.00 -> 157.7 mm, vias 0 -> 1
- net R2: track 0.00 -> 155.5 mm
- net A2: track 0.00 -> 154.2 mm
- net Net-(D10-DIN): track 0.00 -> 144.7 mm
- net OLED SCL: track 0.00 -> 142.0 mm
- net OLED SDA: track 0.00 -> 137.8 mm
- net A1: track 0.00 -> 134.0 mm
- net R1: track 0.00 -> 129.6 mm
- net DOWN: track 0.00 -> 124.9 mm
- net B2: track 0.00 -> 120.8 mm
- net L3: track 0.00 -> 120.2 mm
- net R3: track 0.00 -> 119.4 mm
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- added copper zone on B.Cu, net GND
Other:
- board size 11.3 x 21 mm -> 336 x 134 mm
- board text added: "locked"
- board text removed: "A/x/B"
- board text removed: "A1"
- board text removed: "A2"
- board text removed: "B/○/A"
- board text removed: "B1"
- board text removed: "B2"
- board text removed: "B3"
- board text removed: "B4"
- board text removed: "Back/Share/-"
- board text removed: "Down"
- board text removed: "Guide/PS/Home"
- board text removed: "L1"
- board text removed: "L2"
- board text removed: "L3"
- board text removed: "LS/L3/LS"
- board text removed: "LT/L1/L"
- board text removed: "LT/L2/ZL"
- board text removed: "Left"
- board text removed: "NA/Touchpad/Capture"
- board text removed: "R1"
- board text removed: "R2"
- board text removed: "R3"
- board text removed: "RB/R1/R"
- board text removed: "RS/R3/RS"
- board text removed: "RT/R2/ZR"
- board text removed: "Right"
- board text removed: "S1"
- board text removed: "S2"
- board text removed: "Start/Options/+"
- board text removed: "Up"
- board text removed: "X/□/Y"
- board text removed: "Y/△/X"
