File: pcb/genbox.kicad_pcb (KiCad board)
At the start: 2 copper layers, 336 x 134 mm, 60 parts, among them J1 USB_A, SW15 SW_SPST, SW16 SW_SPST, SW17 SW_SPST, SW18 SW_SPST, U1 DM-OLED096-636, U2 rp2040-zero, U3 SN74LV1T34DBV

Commit message: increased OLED hole, enlarged rp2040 pads
Parts:
- U2: footprint mcu:rp2040-zero-tht-pads -> haku:rp2040-zero-tht-pads
Routing:
- net OLED SCL: track 132.0 -> 134.8 mm
- net +5V: track 242.0 -> 243.5 mm
